File: boards/HighPowerDriver/HPDriver/Connector.kicad_sch (KiCad schematic)
At the start: 72 parts, among them J1 60V_In, J2 USB_B_Mini, J3 Coils, J4 Control, Q10 IRF4950S, Q11 BC817, Q12 BC817, Q13 BC817, Q14 BC817, Q9 BC817, SW1 SW_Push, U3 FT230XS, U4 SFH6156, U5 SFH6156, U6 TLP118, U7 LTV-827S, U8 LTV-827S, U9 74HC14

Commit message: Changed Controller to ATmega328PB
The ATtiny did not have enough flash
Parts:
- removed Q11: BC817, Package_TO_SOT_SMD:SOT-23, symbol Transistor_BJT:BC817
- removed R19: 860R, Resistor_SMD:R_0805_2012Metric, symbol Device:R
- removed R25: 330R, Resistor_SMD:R_0805_2012Metric, symbol Device:R
- removed SW1: SW_Push, Button_Switch_SMD:SW_SPST_B3S-1000, symbol Switch:SW_Push
- added D6: LED_Ye, LED_SMD:LED_0805_2012Metric, symbol Device:LED
- added R8: 180R, Resistor_SMD:R_0805_2012Metric, symbol Device:R
- renumbered C29 to C13, C27 to C23, C26 to C29, C25 to C30, C22 to C31, C23 to C32, C24 to C33, C21 to C34, D4 to D10, D5 to D11, D6 to D12, D9 to D13, D15 to D14, D12 to D15, D13 to D16, D16 to D17, D14 to D18, D7 to D3, D10 to D5, D8 to D7, D11 to D9, J1 to J2, J2 to J5, Q12 to Q1, Q9 to Q2, Q14 to Q3, Q13 to Q4, Q10 to Q5, R28 to R11, R13 to R15, R48 to R17, R49 to R18, R14 to R19, R41 to R24, R40 to R25, R37 to R27, R21 to R28, R39 to R30, R15 to R32, R38 to R33, R27 to R34, R29 to R35, R30 to R36, R24 to R37, R31 to R38, R22 to R39, R32 to R40, R34 to R41, R33 to R42, R36 to R43, R35 to R44, R17 to R45, R23 to R46, R16 to R47, R52 to R48, R26 to R6, R20 to R7, R18 to R9, U5 to U10, U7 to U11, U6 to U12, U8 to U13, U3 to U14, U9 to U8, U4 to U9
Connections:
- net +5V: now also R8.1; no longer R9.1
- net GND: now also D3.1 (K)
- net Ready: now also R9.1
- new net: D6.2 (A), R8.2
- new net LocalCtrl: D6.1 (K)
Other:
- moved on the sheet: D10, D3, D5, D7, D9, Q1, Q2, R11, R15, R28, R32, R6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
